File: sfp-board/Science Fair Project.brd (EAGLE design)
At the start: 115.5 x 92.4 mm, 3 parts

Commit message: Board v3
Parts:
- added R1: 100k, rcl:0411/15
- added R2: OPTO_RES, opto-resistor:OPTO_RES
- added WEMOS2: (no value), esp8266modules:WEMOS-D1-MINI
Connections:
- new net N$8: R1.1, R2.1, WEMOS2.A0
- net N$2: now also R1.2, R2.2, WEMOS2.GND; no longer U$1.1, WEMOS1.5V
- net N$6: now also U$1.1, WEMOS1.5V
Routing:
- net N$6: track 0.00 -> 89.7 mm
- net N$8: track 0.00 -> 59.9 mm
- net N$2: track 36.8 -> 51.2 mm
- net N$7: track 56.1 -> 66.5 mm
- net N$5: track 75.4 -> 83.3 mm
- net N$1: track 74.7 -> 76.5 mm
Changed lines of the file:
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@@
 <layer number="48" name="Document" color="7" fill="1" visible="yes" active="yes"/>
 <layer number="49" name="Reference" color="7" fill="1" visible="yes" active="yes"/>
+<layer number="50" name="dxf" color="7" fill="1" visible="no" active="yes"/>
 <layer number="51" name="tDocu" color="7" fill="1" visible="yes" active="yes"/>
 <layer number="52" name="bDocu" color="7" fill="1" visible="yes" active="yes"/>
@@
 <layer number="101" name="Hidden" color="15" fill="1" visible="yes" active="yes"/>
 <layer number="102" name="Changes" color="12" fill="1" visible="yes" active="yes"/>
+<layer number="250" name="Descript" color="3" fill="1" visible="no" active="no"/>
+<layer number="251" name="SMDround" color="12" fill="11" visible="no" active="no"/>
 </layers>
 <board>
@@
 <attribute name="NAME" x="55.88" y="57.15" size="1.4224" layer="25" align="bottom-right"/>
 </element>
+<element name="WEMOS2" library="esp8266modules" package="WEMOS-D1-MINI" value="" x="78.74" y="78.74" smashed="yes">
+<attribute name="NAME" x="91.44" y="60.96" size="1.4224" layer="25" align="bottom-right"/>
+</element>
+<element name="R1" library="rcl" library_urn="urn:adsk.eagle:library:334" package="0411/15" package3d_urn="urn:adsk.eagle:package:23568/1" value="100k" x="106.68" y="60.96" smashed="yes">
+<attribute name="NAME" x="106.68" y="64.643" size="1.27" layer="25" ratio="10"/>
+<attribute name="SPICEPREFIX" value="R" x="106.68" y="60.96" size="1.778" layer="27" display="off"/>
+<attribute name="VALUE" x="103.0986" y="60.325" size="1.27" layer="27" ratio="10"/>
+</element>
+<element name="R2" library="opto-resistor" package="OPTO_RES" value="OPTO_RES" x="120.65" y="78.74" smashed="yes">
+<attribute name="NAME" x="135.89" y="87.63" size="2.1844" layer="25"/>
+<attribute name="VALUE" x="135.89" y="83.82" size="2.1844" layer="27"/>
+</element>
 </elements>
 <signals>
@@
 <contactref element="U$2" pad="2"/>
 <contactref element="U$2" pad="4"/>
-<wire x1="85.344" y1="14.0208" x2="65.6844" y2="14.0208" width="0.1524" layer="1"/>
+<wire x1="84.074" y1="14.0208" x2="65.6844" y2="14.0208" width="0.1524" layer="1"/>
 <wire x1="65.6844" y1="14.0208" x2="55.9308" y2="14.0208" width="0.1524" layer="1"/>
-<wire x1="85.9536" y1="14.6304" x2="85.344" y2="14.0208" width="0.1524" layer="1"/>
-<wire x1="87.0204" y1="14.6304" x2="85.9536" y2="14.6304" width="0.1524" layer="1"/>
-<wire x1="88.8492" y1="12.8016" x2="87.0204" y2="14.6304" width="0.1524" layer="1"/>
+<wire x1="84.6836" y1="14.6304" x2="84.074" y2="14.0208" width="0.1524" layer="1"/>
+<wire x1="87.9348" y1="14.6304" x2="84.6836" y2="14.6304" width="0.1524" layer="1"/>
 <wire x1="55.9308" y1="14.0208" x2="55.88" y2="13.97" width="0.1524" layer="1"/>
-<wire x1="88.8492" y1="12.8016" x2="88.9" y2="12.7" width="0.1524" layer="1"/>
-<wire x1="92.0496" y1="14.6304" x2="93.98" y2="12.7" width="0.1524" layer="16"/>
-<wire x1="90.8304" y1="14.6304" x2="92.0496" y2="14.6304" width="0.1524" layer="16"/>
-<wire x1="88.9" y1="12.7" x2="90.8304" y2="14.6304" width="0.1524" layer="16"/>
+<wire x1="87.9348" y1="14.6304" x2="88.9" y2="12.7" width="0.1524" layer="1"/>
+<wire x1="93.98" y1="13.97" x2="93.98" y2="12.7" width="0.1524" layer="16"/>
+<wire x1="93.98" y1="13.97" x2="93.3196" y2="14.6304" width="0.1524" layer="16"/>
+<wire x1="89.5604" y1="14.6304" x2="93.3196" y2="14.6304" width="0.1524" layer="16"/>
+<wire x1="89.5604" y1="14.6304" x2="88.9" y2="13.97" width="0.1524" layer="16"/>
+<wire x1="88.9" y1="12.7" x2="88.9" y2="13.97" width="0.1524" layer="16"/>
 <wire x1="65.6844" y1="44.8056" x2="63.5" y2="46.99" width="0.1524" layer="1"/>
 <wire x1="65.6844" y1="14.0208" x2="65.6844" y2="44.8056" width="0.1524" layer="1"/>
-</signal>
-<signal name="N$2">
-<contactref element="U$1" pad="1"/>
-<contactref element="WEMOS1" pad="5V"/>
-<wire x1="48.3108" y1="29.2608" x2="48.3108" y2="14.0208" width="0.1524" layer="1"/>
-<wire x1="63.5" y1="44.45" x2="48.3108" y2="29.2608" width="0.1524" layer="1"/>
-<wire x1="48.3108" y1="14.0208" x2="48.26" y2="13.97" width="0.1524" layer="1"/>
 </signal>
 <signal name="N$3">
 <contactref element="U$1" pad="2"/>
 <contactref element="WEMOS1" pad="D0"/>
-<wire x1="50.7492" y1="31.6992" x2="50.7492" y2="14.0208" width="0.1524" layer="16"/>
-<wire x1="38.5572" y1="43.8912" x2="50.7492" y2="31.6992" width="0.1524" layer="16"/>
-<wire x1="38.5572" y1="55.1688" x2="38.5572" y2="43.8912" width="0.1524" layer="16"/>
+<wire x1="43.1292" y1="29.1592" x2="43.1292" y2="21.6408" width="0.1524" layer="16"/>
+<wire x1="38.5572" y1="33.7312" x2="43.1292" y2="29.1592" width="0.1524" layer="16"/>
+<wire x1="38.5572" y1="55.1688" x2="38.5572" y2="33.7312" width="0.1524" layer="16"/>
 <wire x1="40.5384" y1="57.15" x2="38.5572" y2="55.1688" width="0.1524" layer="16"/>
-<wire x1="50.7492" y1="14.0208" x2="50.8" y2="13.97" width="0.1524" layer="16"/>
+<wire x1="43.1292" y1="21.6408" x2="50.8" y2="13.97" width="0.1524" layer="16"/>
 <wire x1="40.5384" y1="57.15" x2="40.64" y2="57.15" width="0.1524" layer="16"/>
 </signal>
@@
 <contactref element="U$2" pad="5"/>
 <contactref element="WEMOS1" pad="A0"/>
-<wire x1="65.9892" y1="43.2816" x2="96.4692" y2="12.8016" width="0.1524" layer="16"/>
-<wire x1="57.15" y1="43.2816" x2="65.9892" y2="43.2816" width="0.1524" layer="16"/>
-<wire x1="40.6908" y1="59.7408" x2="57.15" y2="43.2816" width="0.1524" layer="16"/>
-<wire x1="96.4692" y1="12.8016" x2="96.52" y2="12.7" width="0.1524" layer="16"/>
+<wire x1="58.42" y1="42.0116" x2="84.4042" y2="42.0116" width="0.1524" layer="16"/>
+<wire x1="40.6908" y1="59.7408" x2="58.42" y2="42.0116" width="0.1524" layer="16"/>
+<wire x1="96.52" y1="17.78" x2="96.52" y2="12.7" width="0.1524" layer="16"/>
+<wire x1="96.52" y1="17.78" x2="84.4042" y2="42.0116" width="0.1524" layer="16"/>
 <wire x1="40.6908" y1="59.7408" x2="40.64" y2="59.69" width="0.1524" layer="16"/>
 </signal>
 <signal name="N$6">
 <contactref element="U$2" pad="6"/>
+<contactref element="U$1" pad="1"/>
+<contactref element="WEMOS1" pad="5V"/>
+<wire x1="48.3108" y1="20.3708" x2="48.3108" y2="14.0208" width="0.1524" layer="1"/>
+<wire x1="63.5" y1="44.45" x2="63.5" y2="35.56" width="0.1524" layer="1"/>
+<wire x1="63.5" y1="35.56" x2="48.3108" y2="20.3708" width="0.1524" layer="1"/>
+<wire x1="48.3108" y1="14.0208" x2="48.26" y2="13.97" width="0.1524" layer="1"/>
+<wire x1="97.2312" y1="10.8204" x2="99.06" y2="12.6492" width="0.1524" layer="1"/>
+<wire x1="51.3588" y1="10.8204" x2="97.2312" y2="10.8204" width="0.1524" layer="1"/>
+<wire x1="48.3108" y1="13.8684" x2="51.3588" y2="10.8204" width="0.1524" layer="1"/>
+<wire x1="99.06" y1="12.6492" x2="99.06" y2="12.7" width="0.1524" layer="1"/>
+<wire x1="48.3108" y1="13.8684" x2="48.26" y2="13.97" width="0.1524" layer="1"/>
 </signal>
 <signal name="N$7">
 <contactref element="U$2" pad="3"/>
 <contactref element="WEMOS1" pad="D1"/>
-<wire x1="91.44" y1="29.2608" x2="91.44" y2="12.7" width="0.1524" layer="1"/>
-<wire x1="63.5508" y1="57.15" x2="91.44" y2="29.2608" width="0.1524" layer="1"/>
-<wire x1="63.5508" y1="57.15" x2="63.5" y2="57.15" width="0.1524" layer="1"/>
+<wire x1="91.44" y1="47.0408" x2="91.44" y2="12.7" width="0.1524" layer="1"/>
+<wire x1="81.3308" y1="57.15" x2="91.44" y2="47.0408" width="0.1524" layer="1"/>
+<wire x1="81.3308" y1="57.15" x2="63.5" y2="57.15" width="0.1524" layer="1"/>
+</signal>
+<signal name="N$2">
+<contactref element="WEMOS2" pad="GND"/>
+<contactref element="R2" pad="2"/>
+<contactref element="R1" pad="2"/>
+<wire x1="114.3" y1="62.1792" x2="114.3" y2="60.96" width="0.1524" layer="1"/>
+<wire x1="130.7592" y1="78.6384" x2="114.3" y2="62.1792" width="0.1524" layer="1"/>
+<wire x1="130.7592" y1="78.6384" x2="130.81" y2="78.74" width="0.1524" layer="1"/>
+<wire x1="105.4608" y1="71.0184" x2="91.44" y2="71.0184" width="0.1524" layer="1"/>
+<wire x1="114.3" y1="62.1792" x2="105.4608" y2="71.0184" width="0.1524" layer="1"/>
+<wire x1="91.44" y1="71.0184" x2="91.44" y2="71.12" width="0.1524" layer="1"/>
+</signal>
+<signal name="N$8">
+<contactref element="R1" pad="1"/>
+<contactref element="R2" pad="1"/>
+<contactref element="WEMOS2" pad="A0"/>
+<wire x1="99.06" y1="67.2084" x2="99.06" y2="60.96" width="0.1524" layer="16"/>
+<wire x1="110.49" y1="78.6384" x2="99.06" y2="67.2084" width="0.1524" layer="16"/>
+<wire x1="110.49" y1="78.6384" x2="110.49" y2="78.74" width="0.1524" layer="16"/>
+<wire x1="73.6092" y1="83.82" x2="68.58" y2="83.82" width="0.1524" layer="16"/>
+<wire x1="90.2208" y1="67.2084" x2="73.6092" y2="83.82" width="0.1524" layer="16"/>
+<wire x1="99.06" y1="67.2084" x2="90.2208" y2="67.2084" width="0.1524" layer="16"/>
 </signal>
 </signals>
@@
 which will not be processed correctly with this version.
 </note>
+<note version="8.2" severity="warning">
+Since Version 8.2, EAGLE supports online libraries. The ids
+of those online libraries will not be understood (or retained)
+with this version.
+</note>
+<note version="8.3" severity="warning">
+Since Version 8.3, EAGLE supports URNs for individual library
+assets (packages, symbols, and devices). The URNs of those assets
+will not be understood (or retained) with this version.
+</note>
+<note version="8.3" severity="warning">
+Since Version 8.3, EAGLE supports the association of 3D packages
+with devices in libraries, schematics, and board files. Those 3D
+packages will not be understood (or retained) with this version.
+</note>
 </compatibility>
