File: sfp-board/sfp-board.brd (EAGLE design)
At the start: 115.5 x 92.4 mm, 6 parts

Commit message: Initial version sfp board
Parts:
- added C1: (no value), digital-toy:CAP-PTH-5MM
- added R3: 150ohm, rcl:0411/15
- moved R2 106.0 mm to (15.2, 67.3)
- moved U$2 81.3 mm to (33.0, 6.35)
- moved U$1 47.8 mm to (88.9, 44.5)
- moved WEMOS1 32.4 mm to (64.8, 25.4)
- moved R1 23.6 mm to (87.6, 74.9)
- moved WEMOS2 21.6 mm to (63.5, 63.5)
Connections:
- removed net N$1 (its old number): U$1.4, U$2.2, U$2.4, WEMOS1.GND
- removed net N$2 (its old number): R1.2, R2.2, WEMOS2.GND
- removed net N$6: U$1.1, U$2.6, WEMOS1.5V
- new net GND: C1.2, R2.2, U$1.4, U$2.2, U$2.4, WEMOS1.GND, WEMOS2.GND
- new net VCC: R1.2, R3.1, U$1.1, U$2.6, WEMOS1.5V, WEMOS2.5V
- net N$3: now also U$2.3; no longer U$1.2
- net N$4: now also C1.1, R3.2; no longer WEMOS1.3V3
- net N$7: now also U$1.2; no longer U$2.3
Routing:
- net VCC: track 0.00 -> 152.0 mm, vias 0 -> 2
- net N$6: track 89.7 -> 0.00 mm
- net N$1 (its old number): track 76.5 -> 0.00 mm
- net N$2 (its old number): track 51.2 -> 0.00 mm
- net N$7: track 66.5 -> 23.7 mm
- net N$1: track 83.3 -> 49.5 mm
- net N$2: track 59.9 -> 80.2 mm
- net N$4: track 58.9 -> 43.3 mm
- net N$3: track 49.2 -> 52.8 mm, vias 0 -> 2
- added copper zone on layer 16, net GND
Other:
- board size 115.5 x 92.4 mm -> 100 x 80 mm

Commit message: board V4
Parts:
- removed U$1: TEMP-HUM-SENSOR-DHT11, diy-modules:TEMP-HUM-SENSOR-DHT11
- added S1: DHT11, diy-modules:TEMP-HUM-SENSOR-DHT11
- moved R1 46.2 mm to (41.9, 68.6)
- moved R3 16.9 mm to (26.7, 14.0)
- moved C1 8.03 mm to (22.9, 11.4)
- renumbered U$2 to S2
Connections:
- net GND: now also S1.4; no longer U$1.4
- net N$7: now also S1.2; no longer U$1.2
- net VCC: now also S1.1; no longer U$1.1
Routing:
- net VCC: track 152.0 -> 185.0 mm
- net N$7: track 23.7 -> 54.1 mm
- net N$4: track 43.3 -> 27.0 mm
- net N$2: track 80.2 -> 69.9 mm

Commit message: board v5
Parts:
- C1: value (none) -> capacitor
- R2: value OPTO_RES -> Photoresistor
Routing:
- net N$2: track 69.9 -> 53.7 mm
- net VCC: track 185.0 -> 177.7 mm
Other:
- board size 100 x 80 mm -> 81 x 80 mm
Changed lines of the file:
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@@
 <drawing>
 <settings>
-<setting alwaysvectorfont="no"/>
+<setting alwaysvectorfont="yes"/>
 <setting keepoldvectorfont="yes"/>
 <setting verticaltext="up"/>
@@
 <board>
 <plain>
-<wire x1="0" y1="0" x2="100" y2="0" width="0" layer="20"/>
-<wire x1="100" y1="0" x2="100" y2="80" width="0" layer="20"/>
-<wire x1="100" y1="80" x2="0" y2="80" width="0" layer="20"/>
+<wire x1="0" y1="0" x2="80.95" y2="0" width="0" layer="20"/>
+<wire x1="80.95" y1="0" x2="80.95" y2="80" width="0" layer="20"/>
+<wire x1="80.95" y1="80" x2="0" y2="80" width="0" layer="20"/>
 <wire x1="0" y1="80" x2="0" y2="0" width="0" layer="20"/>
 </plain>
@@
 </autorouter>
 <elements>
-<element name="C1" library="digital-toy" package="CAP-PTH-5MM" value="" x="22.86" y="11.43" smashed="yes" rot="R90">
+<element name="C1" library="digital-toy" package="CAP-PTH-5MM" value="capacitor" x="22.86" y="11.43" smashed="yes" rot="R90">
 <attribute name="NAME" x="21.59" y="10.668" size="0.6096" layer="25" rot="R90"/>
-<attribute name="VALUE" x="24.384" y="10.414" size="0.6096" layer="27" rot="R90"/>
+<attribute name="VALUE" x="21.844" y="12.954" size="0.6096" layer="27" rot="R90"/>
 </element>
 <element name="R1" library="rcl" package="0411/15" value="100k" x="41.91" y="68.58" smashed="yes">
-<attribute name="NAME" x="38.1" y="67.183" size="1.27" layer="25" ratio="10"/>
+<attribute name="NAME" x="43.18" y="69.723" size="1.27" layer="25" ratio="10"/>
 <attribute name="SPICEPREFIX" value="R" x="41.91" y="68.58" size="1.778" layer="27" display="off"/>
-<attribute name="VALUE" x="39.5986" y="69.215" size="1.27" layer="27" ratio="10"/>
-</element>
-<element name="R2" library="opto-resistor" package="OPTO_RES" value="OPTO_RES" x="15.24" y="67.31" smashed="yes">
-<attribute name="NAME" x="30.48" y="76.2" size="2.1844" layer="25"/>
-<attribute name="VALUE" x="30.48" y="72.39" size="2.1844" layer="27"/>
+<attribute name="VALUE" x="42.1386" y="66.675" size="1.27" layer="27" ratio="10"/>
+</element>
+<element name="R2" library="opto-resistor" package="OPTO_RES" value="Photoresistor" x="15.24" y="67.31" smashed="yes">
+<attribute name="NAME" x="24.13" y="76.2" size="2.1844" layer="25"/>
 </element>
 <element name="R3" library="rcl" package="0411/15" value="150ohm" x="26.67" y="13.97" smashed="yes" rot="R270">
 <attribute name="NAME" x="29.083" y="19.05" size="1.27" layer="25" ratio="10" rot="R270"/>
 <attribute name="SPICEPREFIX" value="R" x="26.67" y="13.97" size="1.778" layer="27" rot="R270" display="off"/>
-<attribute name="VALUE" x="24.765" y="17.5514" size="1.27" layer="27" ratio="10" rot="R270"/>
+<attribute name="VALUE" x="28.575" y="15.0114" size="1.27" layer="27" ratio="10" rot="R270"/>
 </element>
 <element name="S1" library="diy-modules" package="TEMP-HUM-SENSOR-DHT11" value="DHT11" x="39.37" y="63.5" smashed="yes">
@@
 <contactref element="R2" pad="1"/>
 <contactref element="WEMOS2" pad="A0"/>
-<wire x1="34.29" y1="68.58" x2="53.34" y2="68.58" width="0.4064" layer="16"/>
-<wire x1="53.34" y1="68.58" x2="29.21" y2="68.58" width="0.4064" layer="16"/>
-<wire x1="29.21" y1="68.58" x2="26.67" y2="71.12" width="0.4064" layer="16"/>
+<wire x1="53.34" y1="68.58" x2="52.07" y2="68.58" width="0.4064" layer="16"/>
+<wire x1="52.07" y1="68.58" x2="50.8" y2="67.31" width="0.4064" layer="16"/>
+<wire x1="50.8" y1="67.31" x2="35.56" y2="67.31" width="0.4064" layer="16"/>
+<wire x1="34.29" y1="68.58" x2="35.56" y2="67.31" width="0.4064" layer="16"/>
+<wire x1="35.56" y1="67.31" x2="30.48" y2="67.31" width="0.4064" layer="16"/>
+<wire x1="30.48" y1="67.31" x2="26.67" y2="71.12" width="0.4064" layer="16"/>
 <wire x1="26.67" y1="71.12" x2="8.89" y2="71.12" width="0.4064" layer="16"/>
 <wire x1="8.89" y1="71.12" x2="5.08" y2="67.31" width="0.4064" layer="16"/>
@@
 <wire x1="50.8" y1="12.7" x2="41.91" y2="21.59" width="0.4064" layer="16"/>
 <wire x1="41.91" y1="21.59" x2="26.67" y2="21.59" width="0.4064" layer="16"/>
-<wire x1="76.2" y1="53.34" x2="60.96" y2="68.58" width="0.4064" layer="16"/>
-<wire x1="60.96" y1="68.58" x2="49.53" y2="68.58" width="0.4064" layer="16"/>
-<wire x1="45.72" y1="53.34" x2="76.2" y2="53.34" width="0.4064" layer="16"/>
+<wire x1="76.2" y1="53.34" x2="73.66" y2="50.8" width="0.4064" layer="16"/>
+<wire x1="73.66" y1="50.8" x2="48.26" y2="50.8" width="0.4064" layer="16"/>
+<wire x1="45.72" y1="53.34" x2="48.26" y2="50.8" width="0.4064" layer="16"/>
 <wire x1="35.56" y1="63.5" x2="45.72" y2="53.34" width="0.4064" layer="16"/>
 <wire x1="25.4" y1="11.43" x2="17.78" y2="11.43" width="0.4064" layer="16"/>
@@
 <wire x1="26.67" y1="12.7" x2="25.4" y2="11.43" width="0.4064" layer="16"/>
 <via x="45.72" y="53.34" extent="1-16" drill="0.6096"/>
-<wire x1="45.72" y1="53.34" x2="41.91" y2="49.53" width="0.254" layer="1"/>
+<wire x1="45.72" y1="53.34" x2="48.26" y2="50.8" width="0.254" layer="1"/>
 <via x="41.91" y="21.59" extent="1-16" drill="0.6096"/>
-<wire x1="41.91" y1="49.53" x2="41.91" y2="21.59" width="0.254" layer="1"/>
+<wire x1="46.99" y1="26.67" x2="41.91" y2="21.59" width="0.254" layer="1"/>
+<wire x1="48.26" y1="50.8" x2="52.07" y2="46.99" width="0.4064" layer="1"/>
+<wire x1="52.07" y1="46.99" x2="52.07" y2="31.75" width="0.4064" layer="1"/>
+<wire x1="52.07" y1="31.75" x2="46.99" y2="26.67" width="0.4064" layer="1"/>
+<wire x1="35.56" y1="63.5" x2="36.83" y2="64.77" width="0.4064" layer="1"/>
+<wire x1="36.83" y1="64.77" x2="49.53" y2="64.77" width="0.4064" layer="1"/>
+<wire x1="49.53" y1="64.77" x2="49.53" y2="68.58" width="0.4064" layer="1"/>
 </signal>
 <signal name="N$1">
@@
 <contactref element="S1" pad="2"/>
 <contactref element="WEMOS1" pad="D1"/>
-<wire x1="38.1" y1="63.5" x2="48.26" y2="53.34" width="0.254" layer="1"/>
-<wire x1="48.26" y1="53.34" x2="49.53" y2="53.34" width="0.254" layer="1"/>
-<wire x1="49.53" y1="53.34" x2="74.93" y2="27.94" width="0.254" layer="1"/>
-<wire x1="74.93" y1="27.94" x2="77.47" y2="27.94" width="0.254" layer="1"/>
+<wire x1="38.1" y1="63.5" x2="73.66" y2="27.94" width="0.254" layer="1"/>
+<wire x1="73.66" y1="27.94" x2="77.47" y2="27.94" width="0.254" layer="1"/>
 </signal>
 </signals>
@@
 <mfgpreviewcolor name="substratecolor" color="0xFF786E46"/>
 </mfgpreviewcolors>
+<errors>
+</errors>
 </board>
 </drawing>

Commit message: boardv6
Parts:
- C1: device digital-toy:CAP-PTH-5MM -> digital-toy:CAP-PTH-LARGE
- moved C1 20.5 mm to (41.9, 19.1), turned to 180 degrees
- moved R3 15.5 mm to (41.9, 11.4), turned to 0 degrees
- moved WEMOS2 5.39 mm to (67.3, 59.7), turned to 180 degrees
Routing:
- net N$7: track 54.1 -> 0.00 mm
- net VCC: track 177.7 -> 123.6 mm, vias 2 -> 0
- net N$2: track 53.7 -> 0.00 mm
- net N$4: track 27.0 -> 54.4 mm
- net N$3: track 52.8 -> 68.1 mm, vias 2 -> 0
- net N$1: track 49.5 -> 47.6 mm, vias 0 -> 2

Commit message: board v7
Parts:
- removed R2: Photoresistor, opto-resistor:OPTO_RES
- added H1, H2, H3, H4: MOUNT-HOLE3.3, holes:3,3
- added R4: Photoresistor, rcl:0411/15
- moved S1 15.7 mm to (54.6, 67.3)
- moved R3 14.2 mm to (39.4, 25.4)
- moved R1 13.3 mm to (54.6, 72.4)
- moved WEMOS1 12.7 mm to (77.5, 25.4)
- moved WEMOS2 12.7 mm to (80.0, 59.7)
- moved S2 7.62 mm to (33.0, 14.0)
- moved C1 3.59 mm to (39.4, 21.6)
Connections:
- net GND: now also R4.1; no longer R2.2
- net N$2: now also R4.2; no longer R2.1
Routing:
- net N$2: track 0.00 -> 71.2 mm
- net N$7: track 0.00 -> 57.6 mm
- net VCC: track 123.6 -> 147.8 mm
- net N$1: track 47.6 -> 66.3 mm, vias 2 -> 0
- net N$4: track 54.4 -> 50.8 mm
- net N$3: track 68.1 -> 65.3 mm, vias 0 -> 1
Other:
- board size 81 x 80 mm -> 107.6 x 80 mm

Commit message: board v8
Parts:
- added LED1: status 2, adafruit:LED5MM
- added LED2: power, adafruit:LED5MM
- added LED3: status 1, adafruit:LED5MM
- added R2: 1k, rcl:0411/15
- added R5, R6: 470, rcl:0411/15
Connections:
- new net N$10: R5.2, WEMOS2.D8
- new net N$5: LED2.A, R2.1
- new net N$6: LED1.A, R5.1
- new net N$8: LED3.A, R6.1
- new net N$9: R6.2, WEMOS1.D8
- net GND: now also LED1.K, LED2.K, LED3.K
- net VCC: now also R2.2
Routing:
- net N$8: track 0.00 -> 72.3 mm
- net N$9: track 0.00 -> 16.8 mm
- net N$10: track 0.00 -> 9.94 mm
- net VCC: track 147.8 -> 153.1 mm
- net N$5: track 0.00 -> 5.08 mm
- net N$6: track 0.00 -> 2.54 mm
- net N$2: track 71.2 -> 69.7 mm
Changed lines of the file:
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@@
 <attribute name="SPICEPREFIX" value="R" x="24.13" y="72.39" size="1.778" layer="27" display="off"/>
+</element>
+<element name="LED1" library="adafruit" package="LED5MM" value="status 2" x="99.06" y="45.72" rot="R270"/>
+<element name="LED2" library="adafruit" package="LED5MM" value="power" x="39.37" y="12.7"/>
+<element name="LED3" library="adafruit" package="LED5MM" value="status 1" x="99.06" y="27.94" rot="R270"/>
+<element name="R2" library="rcl" package="0411/15" value="1k" x="25.4" y="12.7" rot="R180">
+<attribute name="SPICEPREFIX" value="R" x="25.4" y="12.7" size="1.778" layer="27" rot="R180" display="off"/>
+</element>
+<element name="R5" library="rcl" package="0411/15" value="470" x="99.06" y="57.15" rot="R90">
+<attribute name="SPICEPREFIX" value="R" x="99.06" y="57.15" size="1.778" layer="27" rot="R90" display="off"/>
+</element>
+<element name="R6" library="rcl" package="0411/15" value="470" x="57.15" y="11.43">
+<attribute name="SPICEPREFIX" value="R" x="57.15" y="11.43" size="1.778" layer="27" display="off"/>
 </element>
 </elements>
@@
 <wire x1="46.99" y1="72.39" x2="46.99" y2="73.66" width="0.4064" layer="16"/>
 <wire x1="46.99" y1="73.66" x2="49.53" y2="76.2" width="0.4064" layer="16"/>
-<wire x1="49.53" y1="76.2" x2="68.58" y2="76.2" width="0.4064" layer="16"/>
-<wire x1="68.58" y1="76.2" x2="73.66" y2="71.12" width="0.4064" layer="16"/>
-<wire x1="73.66" y1="71.12" x2="73.66" y2="68.58" width="0.4064" layer="16"/>
-<wire x1="73.66" y1="68.58" x2="87.63" y2="54.61" width="0.4064" layer="16"/>
+<wire x1="49.53" y1="76.2" x2="66.04" y2="76.2" width="0.4064" layer="16"/>
+<wire x1="66.04" y1="76.2" x2="87.63" y2="54.61" width="0.4064" layer="16"/>
 <wire x1="87.63" y1="54.61" x2="90.17" y2="54.61" width="0.4064" layer="16"/>
 </signal>
@@
 </polygon>
 <contactref element="R4" pad="1"/>
+<contactref element="LED2" pad="K"/>
+<contactref element="LED3" pad="K"/>
+<contactref element="LED1" pad="K"/>
 </signal>
 <signal name="VCC">
@@
 <wire x1="50.8" y1="35.56" x2="74.93" y2="35.56" width="0.4064" layer="1"/>
 <wire x1="50.8" y1="67.31" x2="50.8" y2="35.56" width="0.4064" layer="1"/>
-<wire x1="62.23" y1="72.39" x2="62.23" y2="69.85" width="0.4064" layer="1"/>
-<wire x1="62.23" y1="69.85" x2="53.34" y2="69.85" width="0.4064" layer="1"/>
+<wire x1="62.23" y1="72.39" x2="60.96" y2="69.85" width="0.4064" layer="1"/>
+<wire x1="60.96" y1="69.85" x2="53.34" y2="69.85" width="0.4064" layer="1"/>
 <wire x1="53.34" y1="69.85" x2="50.8" y2="67.31" width="0.4064" layer="1"/>
 <wire x1="74.93" y1="35.56" x2="85.09" y2="25.4" width="0.4064" layer="1"/>
 <wire x1="85.09" y1="25.4" x2="85.09" y2="15.24" width="0.4064" layer="1"/>
 <wire x1="85.09" y1="15.24" x2="90.17" y2="15.24" width="0.4064" layer="1"/>
+<contactref element="R2" pad="2"/>
+<wire x1="17.78" y1="19.05" x2="17.78" y2="12.7" width="0.4064" layer="16"/>
 </signal>
 <signal name="N$1">
@@
 <wire x1="85.09" y1="27.94" x2="90.17" y2="27.94" width="0.4064" layer="16"/>
 </signal>
+<signal name="N$6">
+<contactref element="LED1" pad="A"/>
+<contactref element="R5" pad="1"/>
+<wire x1="99.06" y1="49.53" x2="99.06" y2="46.99" width="0.4064" layer="16"/>
+</signal>
+<signal name="N$8">
+<contactref element="LED3" pad="A"/>
+<contactref element="R6" pad="1"/>
+<wire x1="49.53" y1="11.43" x2="49.53" y2="7.62" width="0.4064" layer="16"/>
+<wire x1="49.53" y1="7.62" x2="50.8" y2="6.35" width="0.4064" layer="16"/>
+<wire x1="50.8" y1="6.35" x2="88.9" y2="6.35" width="0.4064" layer="16"/>
+<wire x1="88.9" y1="6.35" x2="95.25" y2="12.7" width="0.4064" layer="16"/>
+<wire x1="95.25" y1="12.7" x2="95.25" y2="27.94" width="0.4064" layer="16"/>
+<wire x1="95.25" y1="27.94" x2="96.52" y2="29.21" width="0.4064" layer="16"/>
+<wire x1="96.52" y1="29.21" x2="99.06" y2="29.21" width="0.4064" layer="16"/>
+</signal>
+<signal name="N$5">
+<contactref element="LED2" pad="A"/>
+<contactref element="R2" pad="1"/>
+<wire x1="38.1" y1="12.7" x2="33.02" y2="12.7" width="0.4064" layer="16"/>
+</signal>
+<signal name="N$9">
+<contactref element="WEMOS1" pad="D8"/>
+<contactref element="R6" pad="2"/>
+<wire x1="67.31" y1="17.78" x2="69.85" y2="17.78" width="0.4064" layer="16"/>
+<wire x1="69.85" y1="17.78" x2="72.39" y2="15.24" width="0.4064" layer="16"/>
+<wire x1="72.39" y1="15.24" x2="72.39" y2="12.7" width="0.4064" layer="16"/>
+<wire x1="72.39" y1="12.7" x2="71.12" y2="11.43" width="0.4064" layer="16"/>
+<wire x1="71.12" y1="11.43" x2="64.77" y2="11.43" width="0.4064" layer="16"/>
+</signal>
+<signal name="N$10">
+<contactref element="WEMOS2" pad="D8"/>
+<contactref element="R5" pad="2"/>
+<wire x1="90.17" y1="67.31" x2="96.52" y2="67.31" width="0.4064" layer="16"/>
+<wire x1="96.52" y1="67.31" x2="99.06" y2="64.77" width="0.4064" layer="16"/>
+</signal>
 </signals>

Commit message: board v9
Parts:
- moved R4 1.27 mm to (25.4, 72.4)
- renumbered S2 to GP2Y1010AU0F
Routing:
- net N$2: track 69.7 -> 68.4 mm
Changed lines of the file:
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@@
 <attribute name="VALUE" x="50.8" y="63.5" size="1.27" layer="27" align="top-center"/>
 </element>
-<element name="S2" library="gp2y1010au" package="GP2Y1010AU" value="" x="33.02" y="13.97" smashed="yes"/>
+<element name="GP2Y1010AU0F" library="gp2y1010au" package="GP2Y1010AU" value="" x="33.02" y="13.97" smashed="yes"/>
 <element name="WEMOS1" library="esp8266modules" package="WEMOS-D1-MINI" value="" x="77.47" y="25.4" smashed="yes">
 <attribute name="NAME" x="82.55" y="31.75" size="1.4224" layer="25" align="bottom-right"/>
@@
 <element name="H3" library="holes" package="3,3" value="MOUNT-HOLE3.3" x="99.06" y="7.62"/>
 <element name="H4" library="holes" package="3,3" value="MOUNT-HOLE3.3" x="7.62" y="7.62"/>
-<element name="R4" library="rcl" package="0411/15" value="Photoresistor" x="24.13" y="72.39">
-<attribute name="SPICEPREFIX" value="R" x="24.13" y="72.39" size="1.778" layer="27" display="off"/>
+<element name="R4" library="rcl" package="0411/15" value="Photoresistor" x="25.4" y="72.39" smashed="yes">
+<attribute name="SPICEPREFIX" value="R" x="25.4" y="72.39" size="1.778" layer="27" display="off"/>
+<attribute name="NAME" x="20.32" y="74.803" size="1.27" layer="25" ratio="10"/>
+<attribute name="VALUE" x="20.5486" y="67.945" size="1.27" layer="27" ratio="10"/>
 </element>
 <element name="LED1" library="adafruit" package="LED5MM" value="status 2" x="99.06" y="45.72" rot="R270"/>
@@
 <contactref element="WEMOS2" pad="A0"/>
 <contactref element="R4" pad="2"/>
-<wire x1="31.75" y1="72.39" x2="46.99" y2="72.39" width="0.4064" layer="1"/>
+<wire x1="33.02" y1="72.39" x2="46.99" y2="72.39" width="0.4064" layer="1"/>
 <wire x1="46.99" y1="72.39" x2="46.99" y2="73.66" width="0.4064" layer="16"/>
 <wire x1="46.99" y1="73.66" x2="49.53" y2="76.2" width="0.4064" layer="16"/>
@@
 <contactref element="WEMOS2" pad="GND"/>
 <contactref element="S1" pad="4"/>
-<contactref element="S2" pad="2"/>
+<contactref element="GP2Y1010AU0F" pad="2"/>
 <contactref element="C1" pad="2"/>
 <contactref element="WEMOS1" pad="GND"/>
-<contactref element="S2" pad="4"/>
+<contactref element="GP2Y1010AU0F" pad="4"/>
 <polygon width="0.4064" layer="16" isolate="1.27">
 <vertex x="7.62" y="81.28"/>
@@
 <contactref element="R1" pad="2"/>
 <contactref element="WEMOS2" pad="5V"/>
-<contactref element="S2" pad="6"/>
+<contactref element="GP2Y1010AU0F" pad="6"/>
 <contactref element="WEMOS1" pad="5V"/>
 <contactref element="S1" pad="1"/>
@@
 </signal>
 <signal name="N$1">
-<contactref element="S2" pad="5"/>
+<contactref element="GP2Y1010AU0F" pad="5"/>
 <contactref element="WEMOS1" pad="A0"/>
 <wire x1="15.24" y1="19.05" x2="15.24" y2="17.78" width="0.4064" layer="1"/>
@@
 </signal>
 <signal name="N$3">
-<contactref element="S2" pad="3"/>
+<contactref element="GP2Y1010AU0F" pad="3"/>
 <contactref element="WEMOS1" pad="D0"/>
 <wire x1="10.16" y1="19.05" x2="10.16" y2="26.67" width="0.4064" layer="1"/>
@@
 </signal>
 <signal name="N$4">
-<contactref element="S2" pad="1"/>
+<contactref element="GP2Y1010AU0F" pad="1"/>
 <contactref element="R3" pad="2"/>
 <contactref element="C1" pad="1"/>
@@
 <wire x1="44.196" y1="21.59" x2="44.196" y2="20.066" width="0.4064" layer="16"/>
 <wire x1="44.196" y1="20.066" x2="43.18" y2="19.05" width="0.4064" layer="16"/>
-<wire x1="43.18" y1="19.05" x2="24.13" y2="19.05" width="0.4064" layer="16"/>
-<wire x1="24.13" y1="19.05" x2="20.32" y2="22.86" width="0.4064" layer="16"/>
+<wire x1="43.18" y1="19.05" x2="22.86" y2="19.05" width="0.4064" layer="16"/>
+<wire x1="22.86" y1="19.05" x2="20.32" y2="22.86" width="0.4064" layer="16"/>
 <wire x1="20.32" y1="22.86" x2="7.62" y2="22.86" width="0.4064" layer="16"/>
 <wire x1="7.62" y1="22.86" x2="5.08" y2="20.32" width="0.4064" layer="16"/>
