File: sfp-board/sfp-board.brd (EAGLE design)
At the start: 107.6 x 80 mm, 18 parts

Commit message: board v10
Parts:
- added R7, R9: 10k, rcl:0411/15
Connections:
- new net N$11: R9.1, WEMOS2.D2
- new net N$12: R7.2, WEMOS1.D2
- net GND: now also R9.2
- net VCC: now also R7.1
Routing:
- net N$12: track 0.00 -> 83.2 mm
- net N$11: track 0.00 -> 79.8 mm, vias 0 -> 2
- net VCC: track 153.1 -> 160.8 mm
Changed lines of the file:
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@@
 <layer number="43" name="vRestrict" color="2" fill="10" visible="yes" active="yes"/>
 <layer number="44" name="Drills" color="7" fill="1" visible="no" active="yes"/>
-<layer number="45" name="Holes" color="7" fill="1" visible="yes" active="yes"/>
-<layer number="46" name="Milling" color="3" fill="1" visible="no" active="yes"/>
-<layer number="47" name="Measures" color="7" fill="1" visible="no" active="yes"/>
+<layer number="45" name="Holes" color="7" fill="1" visible="no" active="yes"/>
+<layer number="46" name="Milling" color="3" fill="1" visible="yes" active="yes"/>
+<layer number="47" name="Measures" color="7" fill="1" visible="yes" active="yes"/>
 <layer number="48" name="Document" color="7" fill="1" visible="yes" active="yes"/>
 <layer number="49" name="Reference" color="7" fill="1" visible="yes" active="yes"/>
@@
 <layer number="106" name="bPlate" color="7" fill="1" visible="yes" active="yes"/>
 <layer number="107" name="Crop" color="7" fill="1" visible="yes" active="yes"/>
-<layer number="108" name="fp8" color="7" fill="1" visible="no" active="yes"/>
-<layer number="109" name="fp9" color="7" fill="1" visible="no" active="yes"/>
-<layer number="110" name="fp0" color="7" fill="1" visible="no" active="yes"/>
-<layer number="111" name="LPC17xx" color="7" fill="1" visible="no" active="yes"/>
-<layer number="112" name="tSilk" color="7" fill="1" visible="no" active="yes"/>
+<layer number="108" name="fp8" color="7" fill="1" visible="yes" active="yes"/>
+<layer number="109" name="fp9" color="7" fill="1" visible="yes" active="yes"/>
+<layer number="110" name="fp0" color="7" fill="1" visible="yes" active="yes"/>
+<layer number="111" name="LPC17xx" color="7" fill="1" visible="yes" active="yes"/>
+<layer number="112" name="tSilk" color="7" fill="1" visible="yes" active="yes"/>
 <layer number="113" name="ReferenceLS" color="7" fill="1" visible="no" active="no"/>
 <layer number="116" name="Patch_BOT" color="9" fill="4" visible="yes" active="yes"/>
@@
 <layer number="121" name="_tsilk" color="7" fill="1" visible="yes" active="yes"/>
 <layer number="122" name="_bsilk" color="7" fill="1" visible="yes" active="yes"/>
-<layer number="123" name="tTestmark" color="7" fill="1" visible="no" active="yes"/>
-<layer number="124" name="bTestmark" color="7" fill="1" visible="no" active="yes"/>
-<layer number="125" name="_tNames" color="7" fill="1" visible="no" active="yes"/>
-<layer number="126" name="_bNames" color="7" fill="1" visible="no" active="yes"/>
-<layer number="127" name="_tValues" color="7" fill="1" visible="no" active="yes"/>
-<layer number="128" name="_bValues" color="7" fill="1" visible="no" active="yes"/>
+<layer number="123" name="tTestmark" color="7" fill="1" visible="yes" active="yes"/>
+<layer number="124" name="bTestmark" color="7" fill="1" visible="yes" active="yes"/>
+<layer number="125" name="_tNames" color="7" fill="1" visible="yes" active="yes"/>
+<layer number="126" name="_bNames" color="7" fill="1" visible="yes" active="yes"/>
+<layer number="127" name="_tValues" color="7" fill="1" visible="yes" active="yes"/>
+<layer number="128" name="_bValues" color="7" fill="1" visible="yes" active="yes"/>
 <layer number="129" name="Mask" color="7" fill="1" visible="yes" active="yes"/>
 <layer number="130" name="mbStop" color="7" fill="1" visible="yes" active="yes"/>
-<layer number="131" name="tAdjust" color="7" fill="1" visible="no" active="yes"/>
-<layer number="132" name="bAdjust" color="7" fill="1" visible="no" active="yes"/>
+<layer number="131" name="tAdjust" color="7" fill="1" visible="yes" active="yes"/>
+<layer number="132" name="bAdjust" color="7" fill="1" visible="yes" active="yes"/>
 <layer number="133" name="mtFinish" color="7" fill="1" visible="yes" active="yes"/>
 <layer number="134" name="mbFinish" color="7" fill="1" visible="yes" active="yes"/>
@@
 <layer number="148" name="mDocument" color="7" fill="1" visible="yes" active="yes"/>
 <layer number="149" name="mReference" color="7" fill="1" visible="yes" active="yes"/>
-<layer number="150" name="Notes" color="7" fill="1" visible="no" active="yes"/>
+<layer number="150" name="Notes" color="7" fill="1" visible="yes" active="yes"/>
 <layer number="151" name="HeatSink" color="7" fill="1" visible="yes" active="yes"/>
-<layer number="152" name="_bDocu" color="7" fill="1" visible="no" active="yes"/>
+<layer number="152" name="_bDocu" color="7" fill="1" visible="yes" active="yes"/>
 <layer number="153" name="FabDoc1" color="6" fill="1" visible="no" active="no"/>
 <layer number="154" name="FabDoc2" color="2" fill="1" visible="no" active="no"/>
@@
 <layer number="195" name="mNames" color="7" fill="1" visible="yes" active="yes"/>
 <layer number="196" name="mValues" color="7" fill="1" visible="yes" active="yes"/>
-<layer number="199" name="Contour" color="7" fill="1" visible="no" active="yes"/>
+<layer number="199" name="Contour" color="7" fill="1" visible="yes" active="yes"/>
 <layer number="200" name="200bmp" color="1" fill="10" visible="yes" active="yes"/>
 <layer number="201" name="201bmp" color="2" fill="10" visible="yes" active="yes"/>
@@
 <layer number="232" name="Eagle3D_PG2" color="7" fill="1" visible="no" active="no"/>
 <layer number="233" name="Eagle3D_PG3" color="7" fill="1" visible="no" active="no"/>
-<layer number="248" name="Housing" color="7" fill="1" visible="no" active="yes"/>
-<layer number="249" name="Edge" color="7" fill="1" visible="no" active="yes"/>
+<layer number="248" name="Housing" color="7" fill="1" visible="yes" active="yes"/>
+<layer number="249" name="Edge" color="7" fill="1" visible="yes" active="yes"/>
 <layer number="250" name="Descript" color="3" fill="1" visible="no" active="no"/>
 <layer number="251" name="SMDround" color="12" fill="11" visible="no" active="no"/>
@@
 <attribute name="NAME" x="34.29" y="27.813" size="1.27" layer="25" ratio="10"/>
 <attribute name="SPICEPREFIX" value="R" x="39.37" y="25.4" size="1.778" layer="27" display="off"/>
-<attribute name="VALUE" x="38.3286" y="27.305" size="1.27" layer="27" ratio="10"/>
+<attribute name="VALUE" x="37.0586" y="24.765" size="1.27" layer="27" ratio="10"/>
 </element>
 <element name="S1" library="diy-modules" package="TEMP-HUM-SENSOR-DHT11" value="DHT11" x="54.61" y="67.31" smashed="yes">
@@
 <element name="R6" library="rcl" package="0411/15" value="470" x="57.15" y="11.43">
 <attribute name="SPICEPREFIX" value="R" x="57.15" y="11.43" size="1.778" layer="27" display="off"/>
+</element>
+<element name="R7" library="rcl" package="0411/15" value="10k" x="25.4" y="5.08">
+<attribute name="SPICEPREFIX" value="R" x="25.4" y="5.08" size="1.778" layer="27" display="off"/>
+</element>
+<element name="R9" library="rcl" package="0411/15" value="10k" x="44.45" y="5.08" rot="R180">
+<attribute name="SPICEPREFIX" value="R" x="44.45" y="5.08" size="1.778" layer="27" rot="R180" display="off"/>
 </element>
 </elements>
@@
 <contactref element="LED3" pad="K"/>
 <contactref element="LED1" pad="K"/>
+<contactref element="R9" pad="2"/>
 </signal>
 <signal name="VCC">
@@
 <contactref element="R2" pad="2"/>
 <wire x1="17.78" y1="19.05" x2="17.78" y2="12.7" width="0.4064" layer="16"/>
+<contactref element="R7" pad="1"/>
+<wire x1="17.78" y1="12.7" x2="17.78" y2="5.08" width="0.4064" layer="16"/>
 </signal>
 <signal name="N$1">
@@
 <wire x1="96.52" y1="67.31" x2="99.06" y2="64.77" width="0.4064" layer="16"/>
 </signal>
+<signal name="N$11">
+<contactref element="WEMOS2" pad="D2"/>
+<contactref element="R9" pad="1"/>
+<wire x1="52.07" y1="5.08" x2="69.85" y2="5.08" width="0.4064" layer="1"/>
+<wire x1="69.85" y1="5.08" x2="73.66" y2="7.62" width="0.4064" layer="1"/>
+<wire x1="73.66" y1="7.62" x2="73.66" y2="36.83" width="0.4064" layer="16"/>
+<wire x1="73.66" y1="36.83" x2="73.66" y2="58.42" width="0.4064" layer="1"/>
+<wire x1="73.66" y1="58.42" x2="71.12" y2="59.69" width="0.4064" layer="1"/>
+<wire x1="71.12" y1="59.69" x2="67.31" y2="59.69" width="0.4064" layer="1"/>
+<via x="73.66" y="7.62" extent="1-16" drill="0.6" shape="square"/>
+<via x="73.66" y="36.83" extent="1-16" drill="0.6" shape="square"/>
+</signal>
+<signal name="N$12">
+<contactref element="WEMOS1" pad="D2"/>
+<contactref element="R7" pad="2"/>
+<wire x1="33.02" y1="5.08" x2="35.56" y2="2.54" width="0.4064" layer="1"/>
+<wire x1="35.56" y1="2.54" x2="88.9" y2="2.54" width="0.4064" layer="1"/>
+<wire x1="88.9" y1="2.54" x2="92.71" y2="6.35" width="0.4064" layer="1"/>
+<wire x1="92.71" y1="6.35" x2="92.71" y2="24.13" width="0.4064" layer="1"/>
+<wire x1="92.71" y1="24.13" x2="91.44" y2="25.4" width="0.4064" layer="1"/>
+<wire x1="91.44" y1="25.4" x2="90.17" y2="25.4" width="0.4064" layer="1"/>
+</signal>
 </signals>
