File: sfp-board/sfp-board.brd (EAGLE design)
At the start: 107.6 x 80 mm, 20 parts

Commit message: board with logo & update .gitgnore for ingoring tempoary file
Parts:
- added U$1: BRS-SYMBOL, digital-toy:BRS
Changed lines of the file:
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@@
 <attribute name="SPICEPREFIX" value="R" x="44.45" y="5.08" size="1.778" layer="27" rot="R180" display="off"/>
 </element>
+<element name="U$1" library="digital-toy" package="BRS" value="BRS-SYMBOL" x="1.27" y="43.18"/>
 </elements>
 <signals>

Commit message: Board v13
Parts:
- removed C1: capacitor, digital-toy:CAP-PTH-LARGE
- removed R3: 150ohm, rcl:0411/15
- added JP1: (no value), SparkFun:1X02_LONGPADS
- moved R4 7.62 mm to (33.0, 72.4)
- moved U$1 2.54 mm to (1.27, 45.7)
Connections:
- net GND: now also JP1.2; no longer C1.2
- net N$4: now also GP2Y1010AU0F.6, WEMOS1.3V3; no longer C1.1, R3.2
- net VCC: now also JP1.1; no longer GP2Y1010AU0F.6, R3.1
Routing:
- net VCC: track 160.8 -> 202.1 mm
- net N$4: track 51.3 -> 69.9 mm
- net N$2: track 68.4 -> 60.8 mm
- net N$14: track 66.3 -> 60.5 mm, vias 0 -> 2
- net N$12: track 83.2 -> 85.7 mm

Commit message: board v14 with new dustsensor reader
Parts:
- added C1: 220uF, SparkFun:CPOL-RADIAL-100UF-25V
- added R3: 150, rcl:0411/15
Connections:
- new net N$1: C1.1, GP2Y1010AU0F.1, R3.1
- net GND: now also C1.2
- net N$14: no longer WEMOS1.A0
- net N$4: now also WEMOS1.A0; no longer GP2Y1010AU0F.1, GP2Y1010AU0F.6, WEMOS1.3V3
- net VCC: now also GP2Y1010AU0F.6, R3.2
Routing:
- net N$4: track 69.9 -> 0.00 mm
- net N$1: track 0.00 -> 31.3 mm
- net VCC: track 202.1 -> 212.2 mm
- net N$14: track 60.5 -> 54.2 mm
Changed lines of the file:
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@@
 <element name="U$1" library="digital-toy" package="BRS" value="BRS-SYMBOL" x="1.27" y="45.72"/>
 <element name="JP1" library="SparkFun" package="1X02_LONGPADS" value="" x="20.32" y="73.66" rot="R180"/>
+<element name="C1" library="SparkFun" package="CPOL-RADIAL-100UF-25V" value="220uF" x="24.13" y="19.05" rot="R180"/>
+<element name="R3" library="rcl" package="0411/15" value="150" x="36.83" y="19.05">
+<attribute name="SPICEPREFIX" value="R" x="36.83" y="19.05" size="1.778" layer="27" display="off"/>
+</element>
 </elements>
 <signals>
@@
 <contactref element="WEMOS2" pad="GND"/>
 <contactref element="S1" pad="4"/>
-<contactref element="GP2Y1010AU0F" pad="2"/>
 <contactref element="WEMOS1" pad="GND"/>
 <contactref element="GP2Y1010AU0F" pad="4"/>
@@
 <contactref element="R9" pad="2"/>
 <contactref element="JP1" pad="2"/>
+<contactref element="C1" pad="2"/>
+<contactref element="GP2Y1010AU0F" pad="2"/>
 </signal>
 <signal name="VCC">
@@
 <wire x1="20.32" y1="15.24" x2="46.99" y2="15.24" width="0.4064" layer="1"/>
 <wire x1="46.99" y1="15.24" x2="48.26" y2="16.51" width="0.4064" layer="1"/>
-<wire x1="48.26" y1="16.51" x2="48.26" y2="35.56" width="0.4064" layer="1"/>
+<wire x1="48.26" y1="16.51" x2="48.26" y2="19.05" width="0.4064" layer="1"/>
+<contactref element="GP2Y1010AU0F" pad="6"/>
+<contactref element="R3" pad="2"/>
+<wire x1="48.26" y1="19.05" x2="48.26" y2="35.56" width="0.4064" layer="1"/>
+<wire x1="44.45" y1="19.05" x2="48.26" y2="19.05" width="0.4064" layer="1"/>
+<wire x1="17.78" y1="19.05" x2="17.78" y2="12.7" width="0.4064" layer="16"/>
 </signal>
 <signal name="N$3">
@@
 <wire x1="60.96" y1="26.67" x2="62.23" y2="27.94" width="0.4064" layer="16"/>
 <wire x1="62.23" y1="27.94" x2="67.31" y2="27.94" width="0.4064" layer="16"/>
-</signal>
-<signal name="N$4">
-<contactref element="GP2Y1010AU0F" pad="1"/>
-<contactref element="GP2Y1010AU0F" pad="6"/>
-<contactref element="WEMOS1" pad="3V3"/>
-<wire x1="5.08" y1="19.05" x2="5.08" y2="16.51" width="0.4064" layer="1"/>
-<wire x1="5.08" y1="16.51" x2="6.35" y2="15.24" width="0.4064" layer="1"/>
-<wire x1="6.35" y1="15.24" x2="16.51" y2="15.24" width="0.4064" layer="1"/>
-<wire x1="16.51" y1="15.24" x2="17.78" y2="16.51" width="0.4064" layer="1"/>
-<wire x1="17.78" y1="16.51" x2="17.78" y2="19.05" width="0.4064" layer="1"/>
-<wire x1="17.78" y1="19.05" x2="62.23" y2="19.05" width="0.4064" layer="16"/>
-<wire x1="62.23" y1="19.05" x2="66.04" y2="15.24" width="0.4064" layer="16"/>
-<wire x1="66.04" y1="15.24" x2="67.31" y2="15.24" width="0.4064" layer="16"/>
 </signal>
 <signal name="N$7">
@@
 </signal>
 <signal name="N$14">
-<contactref element="WEMOS1" pad="A0"/>
 <contactref element="GP2Y1010AU0F" pad="5"/>
-<wire x1="67.31" y1="30.48" x2="60.96" y2="30.48" width="0.4064" layer="16"/>
 <wire x1="60.96" y1="30.48" x2="60.96" y2="29.21" width="0.4064" layer="16"/>
 <wire x1="60.96" y1="29.21" x2="59.69" y2="27.94" width="0.4064" layer="16"/>
@@
 <wire x1="15.24" y1="22.86" x2="15.24" y2="19.05" width="0.4064" layer="16"/>
 </signal>
+<signal name="N$1">
+<contactref element="GP2Y1010AU0F" pad="1"/>
+<contactref element="C1" pad="1"/>
+<contactref element="R3" pad="1"/>
+<wire x1="22.86" y1="19.05" x2="22.86" y2="17.78" width="0.4064" layer="1"/>
+<wire x1="22.86" y1="17.78" x2="21.59" y2="16.51" width="0.4064" layer="1"/>
+<wire x1="21.59" y1="16.51" x2="6.35" y2="16.51" width="0.4064" layer="1"/>
+<wire x1="6.35" y1="16.51" x2="5.08" y2="17.78" width="0.4064" layer="1"/>
+<wire x1="5.08" y1="17.78" x2="5.08" y2="19.05" width="0.4064" layer="1"/>
+<wire x1="22.86" y1="19.05" x2="22.86" y2="20.32" width="0.4064" layer="16"/>
+<wire x1="22.86" y1="20.32" x2="24.13" y2="21.59" width="0.4064" layer="16"/>
+<wire x1="24.13" y1="21.59" x2="27.94" y2="21.59" width="0.4064" layer="16"/>
+<wire x1="27.94" y1="21.59" x2="29.21" y2="20.32" width="0.4064" layer="16"/>
+<wire x1="29.21" y1="20.32" x2="29.21" y2="19.05" width="0.4064" layer="16"/>
+</signal>
+<signal name="N$4">
+<contactref element="WEMOS1" pad="A0"/>
+</signal>
 </signals>

Commit message: Board v15
Routing:
- net N$14: track 54.2 -> 0.00 mm, vias 2 -> 0
- net N$7: track 57.6 -> 68.8 mm
Changed lines of the file:
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@@
 <elements>
 <element name="R1" library="rcl" package="0411/15" value="100k" x="54.61" y="72.39" smashed="yes">
-<attribute name="NAME" x="55.88" y="73.533" size="1.27" layer="25" ratio="10"/>
+<attribute name="NAME" x="60.96" y="74.803" size="1.27" layer="25" ratio="10"/>
 <attribute name="SPICEPREFIX" value="R" x="54.61" y="72.39" size="1.778" layer="27" display="off"/>
-<attribute name="VALUE" x="54.8386" y="70.485" size="1.27" layer="27" ratio="10"/>
+<attribute name="VALUE" x="54.8386" y="71.755" size="1.27" layer="27" ratio="10"/>
 </element>
 <element name="S1" library="diy-modules" package="TEMP-HUM-SENSOR-DHT11" value="DHT11" x="54.61" y="67.31" smashed="yes">
-<attribute name="NAME" x="59.69" y="64.77" size="1.27" layer="25" align="bottom-center"/>
-<attribute name="VALUE" x="50.8" y="63.5" size="1.27" layer="27" align="top-center"/>
+<attribute name="NAME" x="62.23" y="66.04" size="1.27" layer="25" align="bottom-center"/>
+<attribute name="VALUE" x="58.42" y="62.23" size="1.27" layer="27" align="top-center"/>
 </element>
 <element name="GP2Y1010AU0F" library="gp2y1010au" package="GP2Y1010AU" value="" x="33.02" y="13.97" smashed="yes"/>
@@
 <contactref element="S1" pad="2"/>
 <contactref element="WEMOS1" pad="D1"/>
-<wire x1="53.34" y1="67.31" x2="53.34" y2="59.69" width="0.4064" layer="16"/>
-<wire x1="53.34" y1="59.69" x2="85.09" y2="27.94" width="0.4064" layer="16"/>
+<wire x1="53.34" y1="67.31" x2="53.34" y2="40.64" width="0.4064" layer="16"/>
+<wire x1="53.34" y1="40.64" x2="54.61" y2="39.37" width="0.4064" layer="16"/>
+<wire x1="54.61" y1="39.37" x2="73.66" y2="39.37" width="0.4064" layer="16"/>
+<wire x1="73.66" y1="39.37" x2="85.09" y2="27.94" width="0.4064" layer="16"/>
 <wire x1="85.09" y1="27.94" x2="90.17" y2="27.94" width="0.4064" layer="16"/>
 </signal>
@@
 <signal name="N$14">
 <contactref element="GP2Y1010AU0F" pad="5"/>
-<wire x1="60.96" y1="30.48" x2="60.96" y2="29.21" width="0.4064" layer="16"/>
-<wire x1="60.96" y1="29.21" x2="59.69" y2="27.94" width="0.4064" layer="16"/>
-<via x="59.69" y="27.94" extent="1-16" drill="0.6" shape="square"/>
-<wire x1="59.69" y1="27.94" x2="59.69" y2="26.67" width="0.4064" layer="1"/>
-<wire x1="59.69" y1="26.67" x2="57.15" y2="24.13" width="0.4064" layer="1"/>
-<wire x1="57.15" y1="24.13" x2="50.8" y2="24.13" width="0.4064" layer="1"/>
-<via x="50.8" y="24.13" extent="1-16" drill="0.6" shape="square"/>
-<wire x1="50.8" y1="24.13" x2="16.51" y2="24.13" width="0.4064" layer="16"/>
-<wire x1="16.51" y1="24.13" x2="15.24" y2="22.86" width="0.4064" layer="16"/>
-<wire x1="15.24" y1="22.86" x2="15.24" y2="19.05" width="0.4064" layer="16"/>
 </signal>
 <signal name="N$1">

Commit message: Board v16 with 4th Gen Code
Parts:
- JP1: value (none) -> POWER
Changed lines of the file:
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@@
 </element>
 <element name="U$1" library="digital-toy" package="BRS" value="BRS-SYMBOL" x="1.27" y="45.72"/>
-<element name="JP1" library="SparkFun" package="1X02_LONGPADS" value="" x="20.32" y="73.66" rot="R180"/>
+<element name="JP1" library="SparkFun" package="1X02_LONGPADS" value="POWER" x="20.32" y="73.66" rot="R180"/>
 <element name="C1" library="SparkFun" package="CPOL-RADIAL-100UF-25V" value="220uF" x="24.13" y="19.05" rot="R180"/>
 <element name="R3" library="rcl" package="0411/15" value="150" x="36.83" y="19.05">
@@
 <wire x1="10.16" y1="26.67" x2="11.43" y2="26.67" width="0.4064" layer="1"/>
 <via x="11.43" y="26.67" extent="1-16" drill="0.6" shape="square"/>
-<wire x1="11.43" y1="26.67" x2="60.96" y2="26.67" width="0.4064" layer="16"/>
-<wire x1="60.96" y1="26.67" x2="62.23" y2="27.94" width="0.4064" layer="16"/>
-<wire x1="62.23" y1="27.94" x2="67.31" y2="27.94" width="0.4064" layer="16"/>
+<wire x1="11.43" y1="26.67" x2="64.77" y2="26.67" width="0.4064" layer="16"/>
+<wire x1="64.77" y1="26.67" x2="66.04" y2="27.94" width="0.4064" layer="16"/>
+<wire x1="66.04" y1="27.94" x2="67.31" y2="27.94" width="0.4064" layer="16"/>
 </signal>
 <signal name="N$7">

Commit message: Board v17
Connections:
- removed net N$14: GP2Y1010AU0F.5
- net N$4: now also GP2Y1010AU0F.5
Routing:
- net N$4: track 0.00 -> 62.0 mm, vias 0 -> 2
Changed lines of the file:
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@@
 <wire x1="93.98" y1="25.4" x2="90.17" y2="25.4" width="0.4064" layer="1"/>
-</signal>
-<signal name="N$14">
-<contactref element="GP2Y1010AU0F" pad="5"/>
 </signal>
 <signal name="N$1">
@@
 </signal>
 <signal name="N$4">
+<contactref element="GP2Y1010AU0F" pad="5"/>
 <contactref element="WEMOS1" pad="A0"/>
+<wire x1="15.24" y1="19.05" x2="15.24" y2="22.86" width="0.4064" layer="16"/>
+<wire x1="15.24" y1="22.86" x2="16.51" y2="24.13" width="0.4064" layer="16"/>
+<wire x1="16.51" y1="24.13" x2="44.45" y2="24.13" width="0.4064" layer="16"/>
+<wire x1="44.45" y1="24.13" x2="44.45" y2="29.21" width="0.4064" layer="1"/>
+<wire x1="44.45" y1="29.21" x2="63.5" y2="29.21" width="0.4064" layer="16"/>
+<wire x1="63.5" y1="29.21" x2="64.77" y2="30.48" width="0.4064" layer="16"/>
+<wire x1="64.77" y1="30.48" x2="67.31" y2="30.48" width="0.4064" layer="16"/>
+<via x="44.45" y="24.13" extent="1-16" drill="0.6" shape="square"/>
+<via x="44.45" y="29.21" extent="1-16" drill="0.6" shape="square"/>
 </signal>
 </signals>

Commit message: board v18
Parts:
- R4: device rcl:0411/15 -> rcl:0411V
- moved LED2 68.2 mm to (99.1, 45.7), turned to 270 degrees
- moved R4 68.1 mm to (99.1, 55.9), turned to 270 degrees
- moved R5 38.6 mm to (61.0, 50.8)
- moved R7 29.3 mm to (54.6, 7.62)
- moved R9 24.5 mm to (53.3, 27.9), turned to 270 degrees
- moved R1 21.6 mm to (53.3, 50.8), turned to 90 degrees
- moved S1 20.7 mm to (34.3, 71.1), turned to 270 degrees
- moved R2 13.5 mm to (35.6, 21.6)
- moved R3 11.5 mm to (35.6, 7.62)
- moved C1 10.9 mm to (20.3, 8.89), turned to 270 degrees
- moved LED1 10.2 mm to (99.1, 35.6)
- moved R6 4.58 mm to (54.6, 15.2), turned to 180 degrees
- moved LED3 2.54 mm to (99.1, 25.4)
- moved JP1 1.27 mm to (20.3, 72.4)
Routing:
- net GND: track 0.00 -> 71.1 mm, vias 0 -> 1
- net N$5: track 5.08 -> 69.4 mm, vias 0 -> 1
- net N$12: track 85.7 -> 35.3 mm
- net N$11: track 80.0 -> 35.7 mm, vias 2 -> 0
- net N$6: track 2.54 -> 42.2 mm, vias 0 -> 2
- net N$10: track 9.94 -> 44.4 mm
- net N$7: track 68.8 -> 98.7 mm
- net N$3: track 65.3 -> 84.3 mm, vias 1 -> 0
- net N$8: track 72.3 -> 55.0 mm
- net VCC: track 212.2 -> 227.5 mm
- net N$2: track 60.8 -> 51.9 mm
- net N$9: track 16.8 -> 22.1 mm
- net N$4: track 62.0 -> 57.5 mm, vias 2 -> 0
- net N$1: track 31.3 -> 29.1 mm
