File: sfp-board/sfp-board.sch (EAGLE design)
At the start: 6 parts

Commit message: Initial version sfp board
Parts:
- added C1: (no value), digital-toy:CAPPTH1
- added R3: 150ohm, rcl:R-US_0411/15
Connections:
- removed net N$1 (its old number): U$1.GND, U$2.LED-GND, U$2.S-GND, WEMOS1.GND
- removed net N$2 (its old number): R1.2, R2.P2, WEMOS2.GND
- removed net N$6: U$1.VDD, U$2.VCC, WEMOS1.5V
- new net GND: C1.2, R2.P2, U$1.GND, U$2.LED-GND, U$2.S-GND, WEMOS1.GND, WEMOS2.GND
- new net VCC: R1.2, R3.1, U$1.VDD, U$2.VCC, WEMOS1.5V, WEMOS2.5V
- net N$3: now also U$2.LED; no longer U$1.DAT
- net N$4: now also C1.1, R3.2; no longer WEMOS1.3V3
- net N$7: now also U$1.DAT; no longer U$2.LED
Other:
- moved on the sheet: R1, R2, U$1, WEMOS1, WEMOS2

Commit message: board V4
Parts:
- S1: value TEMP-HUM-SENSOR-DHT11 -> DHT11
- renumbered U$1 to S1, U$2 to S2

Commit message: board v5
Parts:
- C1: value (none) -> capacitor
- R2: value OPTO_RES -> Photoresistor
Changed lines of the file:
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@@
 <part name="WEMOS2" library="esp8266modules" deviceset="WEMOS-D1-MINI" device=""/>
 <part name="R1" library="rcl" deviceset="R-US_" device="0411/15" value="100k"/>
-<part name="R2" library="opto-resistor" deviceset="OPTO_RES" device=""/>
+<part name="R2" library="opto-resistor" deviceset="OPTO_RES" device="" value="Photoresistor"/>
 <part name="GND1" library="supply1" deviceset="GND" device=""/>
 <part name="GND2" library="supply1" deviceset="GND" device=""/>
@@
 <part name="R3" library="rcl" deviceset="R-US_" device="0411/15" value="150ohm"/>
 <part name="P+6" library="supply1" deviceset="VCC" device=""/>
-<part name="C1" library="digital-toy" deviceset="CAP" device="PTH1"/>
+<part name="C1" library="digital-toy" deviceset="CAP" device="PTH1" value="capacitor"/>
 </parts>
 <sheets>
@@
 <instance part="C1" gate="G$1" x="-15.24" y="40.64" smashed="yes">
 <attribute name="NAME" x="-17.653" y="39.116" size="1.27" layer="95" rot="R90"/>
-<attribute name="VALUE" x="-11.811" y="38.862" size="1.27" layer="96" rot="R90"/>
+<attribute name="VALUE" x="-11.811" y="41.402" size="1.27" layer="96" rot="R90"/>
 </instance>
 </instances>
@@
 </sheet>
 </sheets>
+<errors>
+</errors>
 </schematic>
 </drawing>

Commit message: boardv6
Parts:
- C1: device digital-toy:CAPPTH1 -> digital-toy:CAPPTH3
Changed lines of the file:
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@@
 <?xml version="1.0" encoding="utf-8"?>
 <!DOCTYPE eagle SYSTEM "eagle.dtd">
-<eagle version="9.2.2">
+<eagle version="7.6.0">
 <drawing>
 <settings>
 <setting alwaysvectorfont="no"/>
-<setting keepoldvectorfont="yes"/>
 <setting verticaltext="up"/>
 </settings>
 <grid distance="0.1" unitdist="inch" unit="inch" style="lines" multiple="1" display="no" altdistance="0.01" altunitdist="inch" altunit="inch"/>
 <layers>
-<layer number="1" name="Top" color="4" fill="1" visible="no" active="no"/>
-<layer number="2" name="Route2" color="1" fill="3" visible="no" active="no"/>
-<layer number="3" name="Route3" color="4" fill="3" visible="no" active="no"/>
-<layer number="4" name="Route4" color="1" fill="4" visible="no" active="no"/>
-<layer number="5" name="Route5" color="4" fill="4" visible="no" active="no"/>
-<layer number="6" name="Route6" color="1" fill="8" visible="no" active="no"/>
-<layer number="7" name="Route7" color="4" fill="8" visible="no" active="no"/>
-<layer number="8" name="Route8" color="1" fill="2" visible="no" active="no"/>
-<layer number="9" name="Route9" color="4" fill="2" visible="no" active="no"/>
-<layer number="10" name="Route10" color="1" fill="7" visible="no" active="no"/>
-<layer number="11" name="Route11" color="4" fill="7" visible="no" active="no"/>
-<layer number="12" name="Route12" color="1" fill="5" visible="no" active="no"/>
-<layer number="13" name="Route13" color="4" fill="5" visible="no" active="no"/>
-<layer number="14" name="Route14" color="1" fill="6" visible="no" active="no"/>
-<layer number="15" name="Route15" color="4" fill="6" visible="no" active="no"/>
-<layer number="16" name="Bottom" color="1" fill="1" visible="no" active="no"/>
-<layer number="17" name="Pads" color="2" fill="1" visible="no" active="no"/>
-<layer number="18" name="Vias" color="2" fill="1" visible="no" active="no"/>
-<layer number="19" name="Unrouted" color="6" fill="1" visible="no" active="no"/>
-<layer number="20" name="Dimension" color="15" fill="1" visible="no" active="no"/>
-<layer number="21" name="tPlace" color="7" fill="1" visible="no" active="no"/>
-<layer number="22" name="bPlace" color="7" fill="1" visible="no" active="no"/>
-<layer number="23" name="tOrigins" color="15" fill="1" visible="no" active="no"/>
-<layer number="24" name="bOrigins" color="15" fill="1" visible="no" active="no"/>
-<layer number="25" name="tNames" color="7" fill="1" visible="no" active="no"/>
-<layer number="26" name="bNames" color="7" fill="1" visible="no" active="no"/>
-<layer number="27" name="tValues" color="7" fill="1" visible="no" active="no"/>
-<layer number="28" name="bValues" color="7" fill="1" visible="no" active="no"/>
+<layer number="1" name="Top" color="4" fill="1" visible="yes" active="no"/>
+<layer number="2" name="Route2" color="1" fill="3" visible="yes" active="no"/>
+<layer number="3" name="Route3" color="4" fill="3" visible="yes" active="no"/>
+<layer number="4" name="Route4" color="1" fill="4" visible="yes" active="no"/>
+<layer number="5" name="Route5" color="4" fill="4" visible="yes" active="no"/>
+<layer number="6" name="Route6" color="1" fill="8" visible="yes" active="no"/>
+<layer number="7" name="Route7" color="4" fill="8" visible="yes" active="no"/>
+<layer number="8" name="Route8" color="1" fill="2" visible="yes" active="no"/>
+<layer number="9" name="Route9" color="4" fill="2" visible="yes" active="no"/>
+<layer number="10" name="Route10" color="1" fill="7" visible="yes" active="no"/>
+<layer number="11" name="Route11" color="4" fill="7" visible="yes" active="no"/>
+<layer number="12" name="Route12" color="1" fill="5" visible="yes" active="no"/>
+<layer number="13" name="Route13" color="4" fill="5" visible="yes" active="no"/>
+<layer number="14" name="Route14" color="1" fill="6" visible="yes" active="no"/>
+<layer number="15" name="Route15" color="4" fill="6" visible="yes" active="no"/>
+<layer number="16" name="Bottom" color="1" fill="1" visible="yes" active="no"/>
+<layer number="17" name="Pads" color="2" fill="1" visible="yes" active="no"/>
+<layer number="18" name="Vias" color="2" fill="1" visible="yes" active="no"/>
+<layer number="19" name="Unrouted" color="6" fill="1" visible="yes" active="no"/>
+<layer number="20" name="Dimension" color="15" fill="1" visible="yes" active="no"/>
+<layer number="21" name="tPlace" color="7" fill="1" visible="yes" active="no"/>
+<layer number="22" name="bPlace" color="7" fill="1" visible="yes" active="no"/>
+<layer number="23" name="tOrigins" color="15" fill="1" visible="yes" active="no"/>
+<layer number="24" name="bOrigins" color="15" fill="1" visible="yes" active="no"/>
+<layer number="25" name="tNames" color="7" fill="1" visible="yes" active="no"/>
+<layer number="26" name="bNames" color="7" fill="1" visible="yes" active="no"/>
+<layer number="27" name="tValues" color="7" fill="1" visible="yes" active="no"/>
+<layer number="28" name="bValues" color="7" fill="1" visible="yes" active="no"/>
 <layer number="29" name="tStop" color="7" fill="3" visible="no" active="no"/>
 <layer number="30" name="bStop" color="7" fill="6" visible="no" active="no"/>
@@
 <layer number="35" name="tGlue" color="7" fill="4" visible="no" active="no"/>
 <layer number="36" name="bGlue" color="7" fill="5" visible="no" active="no"/>
-<layer number="37" name="tTest" color="7" fill="1" visible="no" active="no"/>
-<layer number="38" name="bTest" color="7" fill="1" visible="no" active="no"/>
+<layer number="37" name="tTest" color="7" fill="1" visible="yes" active="no"/>
+<layer number="38" name="bTest" color="7" fill="1" visible="yes" active="no"/>
 <layer number="39" name="tKeepout" color="4" fill="11" visible="no" active="no"/>
 <layer number="40" name="bKeepout" color="1" fill="11" visible="no" active="no"/>
@@
 <layer number="44" name="Drills" color="7" fill="1" visible="no" active="no"/>
 <layer number="45" name="Holes" color="7" fill="1" visible="no" active="no"/>
-<layer number="46" name="Milling" color="3" fill="1" visible="no" active="no"/>
-<layer number="47" name="Measures" color="7" fill="1" visible="no" active="no"/>
-<layer number="48" name="Document" color="7" fill="1" visible="no" active="no"/>
-<layer number="49" name="Reference" color="7" fill="1" visible="no" active="no"/>
-<layer number="50" name="dxf" color="7" fill="1" visible="no" active="no"/>
-<layer number="51" name="tDocu" color="7" fill="1" visible="no" active="no"/>
-<layer number="52" name="bDocu" color="7" fill="1" visible="no" active="no"/>
-<layer number="53" name="tGND_GNDA" color="7" fill="9" visible="no" active="no"/>
-<layer number="54" name="bGND_GNDA" color="1" fill="9" visible="no" active="no"/>
-<layer number="56" name="wert" color="7" fill="1" visible="no" active="no"/>
-<layer number="57" name="tCAD" color="7" fill="1" visible="no" active="no"/>
-<layer number="59" name="tCarbon" color="7" fill="1" visible="no" active="no"/>
-<layer number="60" name="bCarbon" color="7" fill="1" visible="no" active="no"/>
+<layer number="46" name="Milling" color="3" fill="1" visible="yes" active="no"/>
+<layer number="47" name="Measures" color="7" fill="1" visible="yes" active="no"/>
+<layer number="48" name="Document" color="7" fill="1" visible="yes" active="no"/>
+<layer number="49" name="Reference" color="7" fill="1" visible="yes" active="no"/>
+<layer number="50" name="dxf" color="7" fill="1" visible="yes" active="no"/>
+<layer number="51" name="tDocu" color="7" fill="1" visible="yes" active="no"/>
+<layer number="52" name="bDocu" color="7" fill="1" visible="yes" active="no"/>
+<layer number="53" name="tGND_GNDA" color="7" fill="9" visible="yes" active="no"/>
+<layer number="54" name="bGND_GNDA" color="1" fill="9" visible="yes" active="no"/>
+<layer number="56" name="wert" color="7" fill="1" visible="yes" active="no"/>
+<layer number="57" name="tCAD" color="7" fill="1" visible="yes" active="no"/>
+<layer number="59" name="tCarbon" color="7" fill="1" visible="yes" active="no"/>
+<layer number="60" name="bCarbon" color="7" fill="1" visible="yes" active="no"/>
 <layer number="88" name="SimResults" color="9" fill="1" visible="yes" active="yes"/>
 <layer number="89" name="SimProbes" color="9" fill="1" visible="yes" active="yes"/>
@@
 <part name="R3" library="rcl" deviceset="R-US_" device="0411/15" value="150ohm"/>
 <part name="P+6" library="supply1" deviceset="VCC" device=""/>
-<part name="C1" library="digital-toy" deviceset="CAP" device="PTH1" value="capacitor"/>
+<part name="C1" library="digital-toy" deviceset="CAP" device="PTH3" value="capacitor"/>
 </parts>
 <sheets>

Commit message: board v7
Parts:
- removed R2: Photoresistor, opto-resistor:OPTO_RES
- added H1, H2, H3, H4: MOUNT-HOLE3.3, holes:MOUNT-HOLE3.3
- added R4: Photoresistor, rcl:R-US_0411/15
Connections:
- net GND: now also R4.1; no longer R2.P2
- net N$2: now also R4.2; no longer R2.P1
Changed lines of the file:
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@@
 <part name="WEMOS2" library="esp8266modules" deviceset="WEMOS-D1-MINI" device=""/>
 <part name="R1" library="rcl" deviceset="R-US_" device="0411/15" value="100k"/>
-<part name="R2" library="opto-resistor" deviceset="OPTO_RES" device="" value="Photoresistor"/>
 <part name="GND1" library="supply1" deviceset="GND" device=""/>
 <part name="GND2" library="supply1" deviceset="GND" device=""/>
@@
 <part name="P+6" library="supply1" deviceset="VCC" device=""/>
 <part name="C1" library="digital-toy" deviceset="CAP" device="PTH3" value="capacitor"/>
+<part name="H1" library="holes" deviceset="MOUNT-HOLE" device="3.3"/>
+<part name="H2" library="holes" deviceset="MOUNT-HOLE" device="3.3"/>
+<part name="H3" library="holes" deviceset="MOUNT-HOLE" device="3.3"/>
+<part name="H4" library="holes" deviceset="MOUNT-HOLE" device="3.3"/>
+<part name="R4" library="rcl" deviceset="R-US_" device="0411/15" value="Photoresistor"/>
 </parts>
 <sheets>
@@
 <attribute name="VALUE" x="-24.638" y="100.33" size="1.778" layer="96" rot="R90"/>
 </instance>
-<instance part="R2" gate="G$1" x="-27.94" y="71.12" smashed="yes" rot="R270">
-<attribute name="NAME" x="-33.02" y="82.55" size="1.6764" layer="95" rot="R270"/>
-<attribute name="VALUE" x="-22.86" y="91.44" size="1.4224" layer="96" rot="R270"/>
-</instance>
-<instance part="GND1" gate="1" x="-27.94" y="63.5" smashed="yes">
-<attribute name="VALUE" x="-30.48" y="60.96" size="1.778" layer="96"/>
+<instance part="GND1" gate="1" x="-27.94" y="76.2" smashed="yes">
+<attribute name="VALUE" x="-30.48" y="73.66" size="1.778" layer="96"/>
 </instance>
 <instance part="GND2" gate="1" x="35.56" y="27.94" smashed="yes" rot="R90">
@@
 <attribute name="VALUE" x="-11.811" y="41.402" size="1.27" layer="96" rot="R90"/>
 </instance>
+<instance part="H1" gate="G$1" x="55.88" y="106.68"/>
+<instance part="H2" gate="G$1" x="55.88" y="96.52"/>
+<instance part="H3" gate="G$1" x="58.42" y="86.36"/>
+<instance part="H4" gate="G$1" x="58.42" y="76.2"/>
+<instance part="R4" gate="G$1" x="-27.94" y="86.36" smashed="yes" rot="R90">
+<attribute name="NAME" x="-29.4386" y="87.63" size="1.778" layer="95" rot="R90"/>
+<attribute name="VALUE" x="-24.638" y="80.01" size="1.778" layer="96" rot="R90"/>
+</instance>
 </instances>
 <busses>
@@
 <segment>
 <pinref part="R1" gate="G$1" pin="1"/>
-<pinref part="R2" gate="G$1" pin="P1"/>
 <wire x1="-27.94" y1="91.44" x2="-27.94" y2="93.98" width="0.1524" layer="91"/>
 <pinref part="WEMOS2" gate="D1" pin="A0"/>
@@
 <wire x1="-12.7" y1="93.98" x2="-27.94" y2="93.98" width="0.1524" layer="91"/>
 <junction x="-27.94" y="93.98"/>
+<pinref part="R4" gate="G$1" pin="2"/>
 </segment>
 </net>
 <net name="GND" class="0">
-<segment>
-<pinref part="R2" gate="G$1" pin="P2"/>
-<pinref part="GND1" gate="1" pin="GND"/>
-<wire x1="-27.94" y1="68.58" x2="-27.94" y2="66.04" width="0.1524" layer="91"/>
-</segment>
 <segment>
 <pinref part="WEMOS2" gate="D1" pin="GND"/>
@@
 <wire x1="-15.24" y1="27.94" x2="-22.86" y2="27.94" width="0.1524" layer="91"/>
 </segment>
+<segment>
+<pinref part="R4" gate="G$1" pin="1"/>
+<pinref part="GND1" gate="1" pin="GND"/>
+<wire x1="-27.94" y1="78.74" x2="-27.94" y2="81.28" width="0.1524" layer="91"/>
+</segment>
 </net>

Commit message: board v8
Parts:
- added LED1: status 2, adafruit:LED5MM
- added LED2: power, adafruit:LED5MM
- added LED3: status 1, adafruit:LED5MM
- added R2: 1k, rcl:R-US_0411/15
- added R5, R6: 470, rcl:R-US_0411/15
Connections:
- new net N$10: R5.2, WEMOS2.D8
- new net N$5: LED2.A, R2.1
- new net N$6: LED1.A, R5.1
- new net N$8: LED3.A, R6.1
- new net N$9: R6.2, WEMOS1.D8
- net GND: now also LED1.C, LED2.C, LED3.C
- net VCC: now also R2.2

Commit message: board v9
Parts:
- renumbered S2 to GP2Y1010AU0F
Changed lines of the file:
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@@
 <part name="S1" library="diy-modules" deviceset="TEMP-HUM-SENSOR-DHT11" device="" value="DHT11"/>
 <part name="WEMOS1" library="esp8266modules" deviceset="WEMOS-D1-MINI" device=""/>
-<part name="S2" library="gp2y1010au" deviceset="GP2Y1010AU" device=""/>
+<part name="GP2Y1010AU0F" library="gp2y1010au" deviceset="GP2Y1010AU" device=""/>
 <part name="WEMOS2" library="esp8266modules" deviceset="WEMOS-D1-MINI" device=""/>
 <part name="R1" library="rcl" deviceset="R-US_" device="0411/15" value="100k"/>
@@
 <attribute name="VALUE" x="5.08" y="17.78" size="1.778" layer="96"/>
 </instance>
-<instance part="S2" gate="G$1" x="-7.62" y="25.4" smashed="yes"/>
+<instance part="GP2Y1010AU0F" gate="G$1" x="-7.62" y="25.4" smashed="yes"/>
 <instance part="WEMOS2" gate="D1" x="2.54" y="86.36" smashed="yes">
 <attribute name="NAME" x="-7.62" y="101.6" size="1.778" layer="95"/>
@@
 </segment>
 <segment>
-<pinref part="S2" gate="G$1" pin="LED-GND"/>
+<pinref part="GP2Y1010AU0F" gate="G$1" pin="LED-GND"/>
 <pinref part="GND4" gate="1" pin="GND"/>
 <wire x1="-15.24" y1="38.1" x2="-22.86" y2="38.1" width="0.1524" layer="91"/>
@@
 </segment>
 <segment>
-<pinref part="S2" gate="G$1" pin="S-GND"/>
+<pinref part="GP2Y1010AU0F" gate="G$1" pin="S-GND"/>
 <pinref part="GND6" gate="1" pin="GND"/>
 <wire x1="-15.24" y1="27.94" x2="-22.86" y2="27.94" width="0.1524" layer="91"/>
@@
 </segment>
 <segment>
-<pinref part="S2" gate="G$1" pin="VCC"/>
+<pinref part="GP2Y1010AU0F" gate="G$1" pin="VCC"/>
 <pinref part="P+3" gate="VCC" pin="VCC"/>
 <wire x1="-12.7" y1="17.78" x2="-22.86" y2="17.78" width="0.1524" layer="91"/>
@@
 <net name="N$1" class="0">
 <segment>
-<pinref part="S2" gate="G$1" pin="VOUT"/>
+<pinref part="GP2Y1010AU0F" gate="G$1" pin="VOUT"/>
 <wire x1="-22.86" y1="22.86" x2="-7.62" y2="22.86" width="0.1524" layer="91"/>
 <wire x1="-7.62" y1="22.86" x2="-7.62" y2="40.64" width="0.1524" layer="91"/>
@@
 <net name="N$3" class="0">
 <segment>
-<pinref part="S2" gate="G$1" pin="LED"/>
+<pinref part="GP2Y1010AU0F" gate="G$1" pin="LED"/>
 <wire x1="-22.86" y1="33.02" x2="-5.08" y2="33.02" width="0.1524" layer="91"/>
 <wire x1="-5.08" y1="33.02" x2="-5.08" y2="38.1" width="0.1524" layer="91"/>
@@
 <net name="N$4" class="0">
 <segment>
-<pinref part="S2" gate="G$1" pin="V-LED"/>
+<pinref part="GP2Y1010AU0F" gate="G$1" pin="V-LED"/>
 <wire x1="-22.86" y1="43.18" x2="-20.32" y2="43.18" width="0.1524" layer="91"/>
 <pinref part="R3" gate="G$1" pin="2"/>

Commit message: board v10
Parts:
- added R7, R9: 10k, rcl:R-US_0411/15
Connections:
- new net N$11: R9.1, WEMOS2.D2
- new net N$12: R7.2, WEMOS1.D2
- net GND: now also R9.2
- net VCC: now also R7.1
Changed lines of the file:
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@@
 <part name="GND8" library="supply1" deviceset="GND" device=""/>
 <part name="GND9" library="supply1" deviceset="GND" device=""/>
+<part name="R7" library="rcl" deviceset="R-US_" device="0411/15" value="10k"/>
+<part name="R9" library="rcl" deviceset="R-US_" device="0411/15" value="10k"/>
+<part name="P+8" library="supply1" deviceset="VCC" device=""/>
+<part name="GND10" library="supply1" deviceset="GND" device=""/>
 </parts>
 <sheets>
@@
 <attribute name="VALUE" x="-12.7" y="20.32" size="1.778" layer="96"/>
 </instance>
-<instance part="P+4" gate="VCC" x="33.02" y="25.4" smashed="yes" rot="R270">
-<attribute name="VALUE" x="30.48" y="27.94" size="1.778" layer="96"/>
+<instance part="P+4" gate="VCC" x="35.56" y="25.4" smashed="yes" rot="R270">
+<attribute name="VALUE" x="30.48" y="22.86" size="1.778" layer="96"/>
 </instance>
 <instance part="P+5" gate="VCC" x="45.72" y="33.02" smashed="yes" rot="R90">
@@
 <attribute name="VALUE" x="20.32" y="66.04" size="1.778" layer="96" rot="R90"/>
 </instance>
+<instance part="R7" gate="G$1" x="53.34" y="7.62" smashed="yes" rot="R180">
+<attribute name="NAME" x="52.07" y="6.1214" size="1.778" layer="95" rot="R180"/>
+<attribute name="VALUE" x="54.61" y="10.922" size="1.778" layer="96" rot="R180"/>
+</instance>
+<instance part="R9" gate="G$1" x="35.56" y="88.9" smashed="yes" rot="MR180">
+<attribute name="NAME" x="34.0614" y="85.09" size="1.778" layer="95"/>
+<attribute name="VALUE" x="33.782" y="95.25" size="1.778" layer="96" rot="R180"/>
+</instance>
+<instance part="P+8" gate="VCC" x="60.96" y="7.62" smashed="yes" rot="R270">
+<attribute name="VALUE" x="58.42" y="10.16" size="1.778" layer="96"/>
+</instance>
+<instance part="GND10" gate="1" x="45.72" y="88.9" smashed="yes" rot="R90">
+<attribute name="VALUE" x="48.26" y="86.36" size="1.778" layer="96" rot="R90"/>
+</instance>
 </instances>
 <busses>
@@
 <wire x1="15.24" y1="68.58" x2="12.7" y2="68.58" width="0.1524" layer="91"/>
 </segment>
+<segment>
+<pinref part="R9" gate="G$1" pin="2"/>
+<pinref part="GND10" gate="1" pin="GND"/>
+<wire x1="43.18" y1="88.9" x2="40.64" y2="88.9" width="0.1524" layer="91"/>
+</segment>
 </net>
 <net name="VCC" class="0">
@@
 <pinref part="WEMOS1" gate="D1" pin="5V"/>
 <pinref part="P+4" gate="VCC" pin="VCC"/>
+<wire x1="33.02" y1="25.4" x2="30.48" y2="25.4" width="0.1524" layer="91"/>
 </segment>
 <segment>
@@
 <pinref part="P+7" gate="VCC" pin="VCC"/>
 <wire x1="-45.72" y1="114.3" x2="-45.72" y2="111.76" width="0.1524" layer="91"/>
+</segment>
+<segment>
+<pinref part="R7" gate="G$1" pin="1"/>
+<pinref part="P+8" gate="VCC" pin="VCC"/>
 </segment>
 </net>
@@
 </segment>
 </net>
+<net name="N$11" class="0">
+<segment>
+<pinref part="WEMOS2" gate="D1" pin="D2"/>
+<pinref part="R9" gate="G$1" pin="1"/>
+<wire x1="30.48" y1="88.9" x2="20.32" y2="88.9" width="0.1524" layer="91"/>
+</segment>
+</net>
+<net name="N$12" class="0">
+<segment>
+<pinref part="WEMOS1" gate="D1" pin="D2"/>
+<wire x1="30.48" y1="35.56" x2="33.02" y2="35.56" width="0.1524" layer="91"/>
+<wire x1="33.02" y1="35.56" x2="33.02" y2="33.02" width="0.1524" layer="91"/>
+<wire x1="33.02" y1="33.02" x2="43.18" y2="33.02" width="0.1524" layer="91"/>
+<wire x1="43.18" y1="33.02" x2="43.18" y2="7.62" width="0.1524" layer="91"/>
+<pinref part="R7" gate="G$1" pin="2"/>
+<wire x1="43.18" y1="7.62" x2="48.26" y2="7.62" width="0.1524" layer="91"/>
+</segment>
+</net>
